File: ESP32-C6-WROOM.kicad_pcb (KiCad board)
At the start: 4 copper layers, 50 x 50 mm, 42 parts, among them J1 Conn_01x04, J2 USB_C_Receptacle_USB2.0_16P, J3 Pin 2x5, J4 Pin 2x3, SW1 SW_SPST, SW2 SW_SPST, SW3 SW_SPST, U1 LM1117MP-3.3, U2 HDC3022QDEJRQ1, U3 USBLC6-2SC6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

Commit message: трассировка дорожек
Parts:
- moved R8 6.38 mm to (127.9, 90.3)
- moved D4 2.79 mm to (142.2, 82.0), turned to -90 degrees
- moved C3 2.65 mm to (129.3, 84.0), turned to -90 degrees
- moved C1 0.38 mm to (113.2, 91.9), turned to 180 degrees
- turned F1 to -90 degrees
- turned FB1 to 180 degrees
- turned SW1 to -90 degrees
- turned SW2 to 90 degrees
Routing:
- net +3V3: track 5.50 -> 88.4 mm, vias 0 -> 2
- net Net-(D1-BK): track 0.00 -> 8.71 mm
- net /ESP_EN: track 0.00 -> 8.34 mm
- net Net-(D1-GK): track 0.00 -> 8.25 mm
- net /USER_SW: track 0.00 -> 7.78 mm
- net +5V: track 0.00 -> 7.68 mm
- net Net-(F1-Pad1): track 0.00 -> 6.28 mm
- net /BOOT9: track 0.00 -> 4.82 mm
- net Net-(D1-RK): track 0.00 -> 4.58 mm
- net /R_LED: track 0.00 -> 4.49 mm, vias 0 -> 1
- net Net-(F1-Pad2): track 0.00 -> 4.26 mm
- net /CC1: track 0.00 -> 3.91 mm
- net Net-(D3-A): track 0.00 -> 3.47 mm
- net /CC2: track 0.00 -> 3.23 mm
- net Net-(U4-GPIO8): track 0.00 -> 2.90 mm
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
Commit message: auto backup
Routing:
- net GNDD: track 5.63 -> 16.2 mm
Changed lines of the file:
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@@
+	)
+	(segment
+		(start 132.004 97.714)
+		(end 132.004 93.904)
+		(width 0.2)
+		(layer "F.Cu")
+		(net 2)
+	)
+	(segment
+		(start 132.004 93.904)
+		(end 131.496 93.904)
+		(width 0.2)
+		(layer "F.Cu")
+		(net 2)
+	)
+	(segment
+		(start 132.512 98.222)
+		(end 132.004 97.714)
+		(width 0.2)
+		(layer "F.Cu")
+		(net 2)
 	)
 	(segment
 		(start 143.16 60.66)
 		(end 143.16 58.11)
+		(width 0.2)
+		(layer "F.Cu")
+		(net 2)
+	)
+	(segment
+		(start 129.34 98.4)
+		(end 132.334 98.4)
+		(width 0.2)
+		(layer "F.Cu")
+		(net 2)
+	)
+	(segment
+		(start 131.18 94.22)
+		(end 129.34 94.22)
 		(width 0.2)
 		(layer "F.Cu")
@@
 	)
 	(segment
+		(start 131.496 93.904)
+		(end 131.18 94.22)
+		(width 0.2)
+		(layer "F.Cu")
+		(net 2)
+	)
+	(segment
 		(start 126.162 86.919)
 		(end 124.13 86.919)
 		(width 0.2)
 		(layer "F.Cu")
+		(net 2)
+	)
+	(segment
+		(start 132.334 98.4)
+		(end 132.512 98.222)
+		(width 0.2)
+		(layer "F.Cu")
